Commit message: Update obstacle avoidance, U-turn, Pure Pursuit analysis and MATLAB response tools

File: src/my_robot_description/urdf/robot.urdf.xacro (robot description, xacro)
@@ -143,6 +143,6 @@
     <parent link="base_link"/>
     <child link="laser_frame"/>
-    <!-- Mounted on top of the chassis, at the front (rotated 180 deg to align heading) -->
-    <origin xyz="0.2 0 ${chassis_height/2 + 0.02}" rpy="0 0 ${pi}"/>
+    <!-- Mounted on top of the chassis, at the front -->
+    <origin xyz="0.2 0 ${chassis_height/2 + 0.02}" rpy="0 0 0"/>
   </joint>
   <!-- IMU Sensor Link & Joint -->

Commit message: Rotate laser_joint 180 deg to fix inverted LiDAR and enable camera by default in real_robot.launch.py

File: src/my_robot_description/urdf/robot.urdf.xacro (robot description, xacro)
@@ -143,6 +143,6 @@
     <parent link="base_link"/>
     <child link="laser_frame"/>
-    <!-- Mounted on top of the chassis, at the front -->
-    <origin xyz="0.2 0 ${chassis_height/2 + 0.02}" rpy="0 0 0"/>
+    <!-- Mounted on top of the chassis, at the front (rotated 180 deg so front aligns with robot front) -->
+    <origin xyz="0.2 0 ${chassis_height/2 + 0.02}" rpy="0 0 ${pi}"/>
   </joint>
   <!-- IMU Sensor Link & Joint -->
